File: Hardware/bGeigieRaku V2.0/M5_board_bGeigieRaku V1.9.5/M5_board_bGeigieRaku V1.9.kicad_pcb (KiCad board)
At the start: 2 copper layers, 129.4 x 64.6 mm, 22 parts, among them J1 M5 2x15 pin, J10 QI GND, J11 QI charger Plus, J2 Geiger, J3 GPS, J4 Conn_01x14_Female, J5 Conn_01x14_Female, J6 Conn_01x14_Female, J7 Conn_01x14_Female, J8 QI charger GND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

Commit message: Updated board V1.9.6
Parts:
- removed J4, J5, J6: Conn_01x14_Female, Connector_PinHeader_2.54mm:PinHeader_1x18_P2.54mm_Vertical
- J1: footprint Connector_PinHeader_2.54mm:PinHeader_2x15_P2.54mm_Vertical -> Connector_PinHeader_2.54mm:PinHeader_2x15_P2.54mm_Vertical_SMD; moved to F.Cu
- J3: footprint Connector_PinHeader_2.54mm:PinHeader_1x04_P2.54mm_Horizontal -> Connector_PinHeader_1.00mm:PinHeader_1x04_P1.00mm_Horizontal
- J7: footprint Connector_PinHeader_2.54mm:PinHeader_1x18_P2.54mm_Vertical -> Connector_PinHeader_2.54mm:PinHeader_1x08_P2.54mm_Vertical
- moved J3 16.3 mm to (158.0, 95.5), turned to 0 degrees
- moved J1 15.8 mm to (123.8, 117.8), turned to -90 degrees
- moved J7 4.39 mm to (155.1, 118.2)
Connections:
- J2 pad 1: GND -> 3.3V
- J2 pad 3: 3.3V -> GND
Routing:
- net GND: track 158.5 -> 16.5 mm, vias 0 -> 3
- net Net-(J1-Pad4): track 88.2 -> 61.8 mm
- net /RX2: track 64.5 -> 43.7 mm, vias 0 -> 1
- net /TX2: track 65.7 -> 45.2 mm, vias 0 -> 1
- net 3.3V: track 126.9 -> 145.0 mm, vias 0 -> 1
- net /SCL: track 64.8 -> 51.8 mm, vias 0 -> 1
- net /Reset: track 94.5 -> 81.9 mm, vias 0 -> 1
- net Net-(J1-Pad30): track 107.8 -> 120.0 mm
- net /TX1: track 52.0 -> 40.3 mm
- net 5V: track 65.9 -> 55.7 mm
- net /SDA: track 60.3 -> 51.0 mm
- net /GIO2: track 99.0 -> 90.8 mm
- net /GIO0: track 75.4 -> 67.7 mm
- net /RX1: track 48.8 -> 41.2 mm
- net /VBATT: track 72.1 -> 73.7 mm
Other:
- board text added: "Safecast M5 based bGeigieRaku prototype board V1.9.6"
- board text removed: "Safecast M5 based bGeigieRaku prototype board V1.9.5"

Commit message: Added pdf of schematic.
Parts:
- J9: value QI Plus -> QI +

Commit message: Fixed board Irover pin reversed
Parts:
- J2: moved to F.Cu
- moved J2 4.61 mm to (207.7, 109.9)
Routing:
- net 3.3V: track 144.8 -> 140.6 mm
