File: Hardware/bGeigieRaku V2.0/M5_board_bGeigieRaku V1.9.5/M5_board_bGeigieRaku V1.9.kicad_pcb (KiCad board)
At the start: 2 copper layers, 129.4 x 64.6 mm, 24 parts, among them J1 M5 2x15 pin, J10 QI GND, J11 QI charger Plus, J2 Geiger, J3 GPS, J7 Conn_01x14_Female, J8 QI charger GND, J9 QI Plus, Q1 ZXMP4A16G, Q2 ZXMP4A16G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

Commit message: added plates and small modifictaions
Parts:
- added D1: DIODE, Diode_THT:D_DO-15_P15.24mm_Horizontal, F.Cu at (160.3, 105.2)
- added D2: DIODE, Diode_THT:D_DO-15_P15.24mm_Horizontal, F.Cu at (165.5, 105.2)
- added G***: LOGO, Symbol:Safecast logo very small, F.Cu at (91.6, 89.1)
- added H11: MountingHole_Pad, MountingHole:MountingHole_3.2mm_M3, F.Cu at (172.3, 125.9)
- added H5: MountingHole_Pad, MountingHole:MountingHole_3.2mm_M3, F.Cu at (208.6, 125.9)
- J3: footprint Connector_PinHeader_1.00mm:PinHeader_1x04_P1.00mm_Horizontal -> Connector_PinSocket_2.54mm:PinSocket_1x04_P2.54mm_Vertical
- J7: footprint Connector_PinHeader_2.54mm:PinHeader_1x18_P2.54mm_Vertical -> Connector_PinHeader_2.54mm:PinHeader_1x10_P2.54mm_Vertical
- Q1, Q2: value ZXMP4A16G -> IRF4905; footprint Package_TO_SOT_SMD:SOT-223-3_TabPin2 -> Package_TO_SOT_THT:TO-220-3_Vertical; moved to B.Cu
- moved Q2 46.0 mm to (157.3, 79.6)
- moved Q1 34.8 mm to (157.3, 73.3)
- moved BT1 2.72 mm to (177.7, 123.0)
- moved H11 1.77 mm to (172.3, 71.8)
- moved H10 1.77 mm to (208.6, 71.8)
- moved J1 1.32 mm to (124.1, 116.5)
- moved H4 1.32 mm to (103.8, 76.8)
- moved H9 1.32 mm to (103.8, 120.8)
- moved H2 0.22 mm to (90.7, 71.8)
- moved H1 0.13 mm to (90.7, 125.9)
- renumbered H5 to H10, H4 to H11, H4 to H9, J2 to J12
Routing:
- net Net-(BT1-Pad1): track 0.00 -> 85.8 mm
- net Net-(D2-Pad1): track 0.00 -> 55.6 mm
- net /TX2: track 12.3 -> 36.7 mm
- net /SCL: track 87.2 -> 83.4 mm
- net /VBATT: track 64.1 -> 67.7 mm, vias 1 -> 0
- net Net-(J1-Pad30): track 110.0 -> 113.6 mm
- net /GIO2: track 103.8 -> 101.9 mm, vias 0 -> 2
- net Net-(J1-Pad4): track 61.2 -> 60.1 mm, vias 1 -> 2
- net /Reset: track 87.1 -> 88.1 mm
- net /RX1: track 71.4 -> 70.6 mm
- net 5V: track 87.8 -> 87.1 mm, vias 1 -> 0
- net /TX1: track 68.1 -> 67.4 mm
- net /SDA: track 78.2 -> 77.8 mm, vias 0 -> 2
Other:
- board text added: "Charge only"
- board text removed: "Battery charger"
- board text removed: "Safecast bGeigieZen board V1.9.6"
