File: Hardware/bGeigieRaku V2.0/M5_board_bGeigieRaku V1.9.5/M5_board_bGeigieRaku V1.9.kicad_pcb (KiCad board)
At the start: 2 copper layers, 129.4 x 64.6 mm, 29 parts, among them J1 M5 2x15 pin, J10 QI GND, J11 QI charger Plus, J12 Geiger, J2 Geiger, J3 GPS, J7 Conn_01x14_Female, J8 QI charger GND, J9 QI Plus, Q1 IRF4905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

Commit message: added logos
Parts:
- removed the G*** at (91.6, 89.1)
- added G***: LOGO, LOGO, F.Cu at (92.6, 99.5)
- added G***: LOGO, bGeigieRaku_M5_1015:18650 map, B.Cu at (178.2, 123.1)
Other:
- board text added: "SDCARD"
- board text added: "USB"
- board text added: "V1.9.6"

Commit message: Update graphics
Parts:
- moved G*** 1.66 mm to (91.1, 100.2)
Changed lines of the file:
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@@
   (net 40 "unconnected-(SW1-Pad1)")
   (footprint "LOGO" (layer "F.Cu")
-    (at 92.6076 99.53 90)
+    (at 91.1076 100.23 90)
     (attr board_only exclude_from_pos_files exclude_from_bom)
     (fp_text reference "G***" (at 0 0 90) (layer "F.SilkS") hide
@@
     (property "Sheetname" "")
     (attr exclude_from_pos_files)
-    (fp_text reference "H5" (at -0.289 -4.939 90) (layer "F.SilkS")
+    (fp_text reference "H5" (at -0.289 -4.939 90) (layer "F.SilkS") hide
       (effects (font (size 1 1) (thickness 0.15)))
     )
@@
     (effects (font (size 1 1) (thickness 0.15)))
   )
-  (gr_text "USB" (at 132.7076 71.63 90) (layer "F.SilkS")
+  (gr_text "USB" (at 126.3076 68.93 180) (layer "F.SilkS")
     (effects (font (size 1.5 1.5) (thickness 0.3)))
   )
@@
     (effects (font (size 0.75 0.75) (thickness 0.15)))
   )
-  (gr_text "SDCARD\n" (at 97.1076 84.93 90) (layer "F.SilkS")
+  (gr_text "SDCARD\n" (at 95.9076 89.93 90) (layer "F.SilkS")
     (effects (font (size 1.5 1.5) (thickness 0.3)))
   )

Commit message: added gerbers for V1.9.6
Other:
- board text added: "GROVE"
- board text added: "bGeigieZen V1.9.6"
Changed lines of the file:
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@@
       (viasonmask false)
       (mode 1)
-      (useauxorigin false)
+      (useauxorigin true)
       (hpglpennumber 1)
       (hpglpenspeed 20)
@@
       (sketchpadsonfab false)
       (subtractmaskfromsilk false)
-      (outputformat 4)
+      (outputformat 1)
       (mirror false)
       (drillshape 0)
       (scaleselection 1)
-      (outputdirectory "gerber 1.9.5/")
+      (outputdirectory "gerber 1.9.6/")
     )
   )
@@
     (effects (font (size 0.75 0.75) (thickness 0.15)) (justify mirror))
   )
+  (gr_text "GROVE" (at 104.6076 69.13 180) (layer "F.SilkS")
+    (effects (font (size 1.5 1.5) (thickness 0.3)))
+  )
   (gr_text "Charge only" (at 212.1326 98.28 90) (layer "F.SilkS")
     (effects (font (size 1 1) (thickness 0.15)))
@@
     (effects (font (size 0.75 0.75) (thickness 0.15)))
   )
+  (gr_text "bGeigieZen\nV1.9.6" (at 196.2076 125.33 180) (layer "F.SilkS")
+    (effects (font (size 1.5 1.5) (thickness 0.3)))
+  )
   (gr_text "ON" (at 174.8536 70.052 90) (layer "F.SilkS")
     (effects (font (size 1.5 1.5) (thickness 0.3)))
@@
         (xy 85.3186 133.298)
         (xy 83.6076 66.43)
-        (xy 214.7176 66.46)
+        (xy 214.2076 66.63)
       )
     )
