File: Hardware/bGeigieRaku V2.0/M5_board_bGeigieRaku V1.9.7/M5_board_bGeigieRaku V1.9.kicad_sch (KiCad schematic)
At the start: 25 parts, among them J1 M5 2x15 pin, J10 QI GND, J11 QI charger Plus, J2 Geiger, J3 GPS, J4 Geiger 2, J5 Extra support header, J8 QI charger GND, J9 QI Plus, Q2 IRFR9024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

Commit message: Updated board to V2.0
Parts:
- Q2: value IRFR9024 -> IRFU9020PBF
Other:
- title: bGeigieZen V1.9.8 -> bGeigieZen V1.2.0
