File: Hardware/bGeigieZen V2.0/bGeigieZen V2.kicad_pcb (KiCad board)
At the start: 2 copper layers, 129.4 x 64.6 mm, 32 parts, among them J1 M5 2x15 pin, J10 QI GND, J11 QI charger Plus, J12 M5 2x15 pin, J2 Geiger, J3 GPS, J4 Geiger 2, J5 Extra support header, J6 Grove, J7 Grove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

Commit message: Updated Board
Parts:
- added G***: LOGO, bGeigieZen:LOGO, F.Cu at (91.1, 100.2)
- added G***: LOGO, bGeigieZen:LOGO, B.Cu at (96.1, 100.3)
- BT1: footprint bGeigieZen:BATTERY_18650-HOLDER -> Library:BATTERY_18650-HOLDER
- R3: footprint bGeigieZen:0207_10 -> bGeigieRaku_M5_1015:0207_10
- sea of pads 1: renamed from REF**
- sea of pads 2: renamed from REF**
- turned J12 to -90 degrees
Connections:
- J1 pad 24: unconnected-(J1-Pin_24) -> Net-(J1-Pin_24)
- J12 pad 1: /BAT -> unconnected-(J12-Pin_1)
- J12 pad 13: unconnected-(J12-Pin_13) -> /SDA
- J12 pad 14: unconnected-(J12-Pin_14) -> /SCL
- J12 pad 20: unconnected-(J12-Pin_20) -> 3.3V
- J12 pad 25: unconnected-(J12-Pin_25) -> GND
- J12 pad 26: GND -> unconnected-(J12-Pin_26)
- J12 pad 27: unconnected-(J12-Pin_27) -> GND
- J12 pad 28: GND -> unconnected-(J12-Pin_28)
- J12 pad 29: unconnected-(J12-Pin_29) -> GND
- J12 pad 30: GND -> unconnected-(J12-Pin_30)
- J12 pad 4: unconnected-(J12-Pin_4) -> Net-(J1-Pin_24)
- J12 pad 6: unconnected-(J12-Pin_6) -> /GIO34
Routing:
- net Net-(J1-Pin_24): track 0.00 -> 59.0 mm
- net /GIO34: track 0.00 -> 44.6 mm
- net /SCL: track 61.6 -> 100.9 mm
- net 3.3V: track 171.4 -> 198.4 mm
- net /BAT: track 156.2 -> 131.8 mm
- net /SDA: track 139.4 -> 156.5 mm
- net GND: track 5.18 -> 11.2 mm, vias 2 -> 1
- net Net-(BT1-+): track 62.8 -> 57.4 mm
- net /GIO2: track 131.3 -> 127.3 mm
- net /RX2: track 49.4 -> 45.6 mm, vias 0 -> 1
- net /TX2: track 49.7 -> 46.0 mm, vias 0 -> 1
- net /Reset: track 92.3 -> 95.1 mm, vias 1 -> 2
- net Net-(J1-Pin_3): track 84.3 -> 86.8 mm, vias 1 -> 2
Other:
- board text added: "Core 2 expansion board"
- board text added: "GPS"
- board text added: "Safepulse"
- board text added: "bGeigieZen V2.1.2 Production"
- board text removed: "bGeigieZen V2.0.2 Production"
