File: Hardware/bGeigieZen V2.0/bGeigieZen V2.kicad_sch (KiCad schematic)
At the start: 29 parts, among them J1 M5 2x15 pin, J10 QI GND, J11 QI charger Plus, J2 Geiger, J3 GPS, J4 Geiger 2, J5 Extra support header, J6 Grove, J7 Grove, J8 QI charger GND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

Commit message: Updated Board
Parts:
- J12: value (none) -> M5 2x15 pin; footprint (none) -> Connector_PinSocket_2.54mm:PinSocket_2x15_P2.54mm_Vertical_SMD
Connections:
- net 3.3V: now also J12.20 (Pin_20)
- net BAT: now also J12.2 (Pin_2); no longer J12.1 (Pin_1)
- net GIO34: now also J12.6 (Pin_6)
- net GND: now also J12.25 (Pin_25), J12.27 (Pin_27), J12.29 (Pin_29); no longer J12.26 (Pin_26), J12.28 (Pin_28), J12.30 (Pin_30)
- net SCL: now also J12.14 (Pin_14)
- net SDA: now also J12.13 (Pin_13)
- net at J1.24 (Pin_24): now also J12.4 (Pin_4)
Other:
- title: bGeigieZen V2.0.2 -> bGeigieZen V2.1.2
- moved on the sheet: J12

Commit message: Changed core2 GIO pins for Geigercounter pulses
Connections:
- net GIO2 renamed GIO2 on Core and GIO32 on Core-2
