File: Hardware/bGeigieZen V3.0.0/bGeigieZen V3.0.0.kicad_sch (KiCad schematic)
At the start: 29 parts, among them J1 M5 2x15 pin, J10 QI GND, J11 QI charger Plus, J12 M5 2x15 pin, J2 Geiger, J3 GPS, J4 Geiger 2, J5 Extra support header, J6 Grove, J7 Grove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

Commit message: board prepared for V3.0.0
Parts:
- removed J12: M5 2x15 pin, Connector_PinSocket_2.54mm:PinSocket_2x15_P2.54mm_Vertical_SMD, symbol Connector_Generic:Conn_02x15_Odd_Even
- removed Q2: IRFU9024N, Package_TO_SOT_THT:TO-251-3_Vertical, symbol IRFR9024:IRFR9024
- removed R1: 9.1k, bGeigieNano V1.1.5:0207_10, symbol Device:R
- removed R2: 1k, bGeigieNano V1.1.5:0207_10, symbol Device:R
- removed R3: 10k, bGeigieRaku_M5_1015:0207_10, symbol Device:R
- J8: value QI charger GND -> QI charger ground
Connections:
- net GND: no longer BT1.2 (-), J8.2 (Pin_2)
- net VBATT: now also BT1.1 (+), J11.1 (Pin_1), J11.2 (Pin_2)
- new net: BT1.2 (-), J8.2 (Pin_2)
Other:
- note added: "QI charger LIPO minus"

Commit message: Updated V3.0.0 board
Parts:
- J11: footprint Connector_PinHeader_2.54mm:PinHeader_1x02_P2.54mm_Vertical -> bGeigieZen:PinHeader_1x02_P2.54mm_Vertical_4056
Changed lines of the file:
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@@
       (effects (font (size 1.27 1.27)) (justify right))
     )
-    (property "Footprint" "Connector_PinHeader_2.54mm:PinHeader_1x02_P2.54mm_Vertical" (at 64.77 80.01 0)
+    (property "Footprint" "bGeigieZen:PinHeader_1x02_P2.54mm_Vertical_4056" (at 64.77 80.01 0)
       (effects (font (size 1.27 1.27)) hide)
     )

Commit message: Cleaned out V3.0.0 board..
Parts:
- removed C1: 47uF, bGeigieNano V1.1.5:C025-024X044, symbol bGeigieRaku-V2-rescue:bGeigieNano_V1.1.5-eagle-import_C-EU025-024X044-bGeigieNa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
- removed H1, H10, H2, H3, H5, H7, H8, H9: MountingHole_Pad, MountingHole:MountingHole_3.2mm_M3, symbol Mechanical:MountingHole_Pad
Connections:
- net Reset: no longer names the net of J1.5 (Pin_5)
Other:
- moved on the sheet: H4, H6
