File: hardware/bGeigieZen V3.0.0/bGeigieZen V3.0.0.kicad_pcb (KiCad board)
At the start: 2 copper layers, 129.4 x 64.6 mm, 18 parts, among them J1 M5 2x15 pin, J10 QI GND, J11 QI charger Plus, J2 Geiger IRover, J3 GPS, J4 Geiger Safepulse, J5 Extra support header, J6 Grove, J8 QI charger ground, J9 QI Plus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

Commit message: Update board layout
Parts:
- moved J10 2.00 mm to (211.8, 91.4)
- moved J11 2.00 mm to (187.1, 104.9)
- moved J8 2.00 mm to (186.5, 91.2)
- moved J9 2.00 mm to (212.0, 105.0)
Routing:
- net /VBATT: track 31.3 -> 63.1 mm
- net Net-(BT1--): track 50.8 -> 52.8 mm
Changed lines of the file:
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@@
   )
   (footprint "Connector_PinHeader_2.54mm:PinHeader_1x02_P2.54mm_Vertical" (layer "F.Cu")
-    (at 209.791904 91.407824 -90)
+    (at 211.791904 91.407824 -90)
     (descr "Through hole straight pin header, 1x02, 2.54mm pitch, single row")
     (tags "Through hole pin header THT 1x02 2.54mm single row")
@@
   )
   (footprint "Connector_PinHeader_2.54mm:PinHeader_1x02_P2.54mm_Vertical" (layer "F.Cu")
-    (at 210.0376 104.977 -90)
+    (at 212.0376 104.977 -90)
     (descr "Through hole straight pin header, 1x02, 2.54mm pitch, single row")
     (tags "Through hole pin header THT 1x02 2.54mm single row")
@@
   )
   (footprint "bGeigieZen:PinHeader_1x02_P2.54mm_Vertical_4056" (layer "F.Cu")
-    (at 185.127021 104.8856 180)
+    (at 187.127021 104.8856 180)
     (descr "Through hole straight pin header, 1x02, 2.54mm pitch, single row")
     (tags "Through hole pin header THT 1x02 2.54mm single row")
@@
   )
   (footprint "Connector_PinHeader_2.54mm:PinHeader_1x02_P2.54mm_Vertical" (layer "F.Cu")
-    (at 184.486504 91.153824)
+    (at 186.486504 91.153824)
     (descr "Through hole straight pin header, 1x02, 2.54mm pitch, single row")
     (tags "Through hole pin header THT 1x02 2.54mm single row")
@@
   (segment (start 128.7526 113.2324) (end 128.7526 116.407) (width 0.5) (layer "B.Cu") (net 4))
   (segment (start 152.883 85.9274) (end 152.883 85.9272) (width 0.5) (layer "B.Cu") (net 4))
-  (segment (start 191.839 112.614) (end 185.127021 105.902021) (width 0.5) (layer "B.Cu") (net 7))
+  (segment (start 188.102811 77.665211) (end 188.102811 100.848753) (width 0.5) (layer "B.Cu") (net 7))
   (segment (start 200.711 117.15) (end 198.78 115.219) (width 0.5) (layer "B.Cu") (net 7))
   (segment (start 207.926 117.15) (end 207.9256 117.15) (width 0.5) (layer "B.Cu") (net 7))
+  (segment (start 197.801 112.614) (end 192.532 112.614) (width 0.5) (layer "B.Cu") (net 7))
   (segment (start 204.4976 117.15) (end 200.711 117.15) (width 0.5) (layer "B.Cu") (net 7))
-  (segment (start 184.3293 73.8917) (end 183.0296 72.592) (width 0.5) (layer "B.Cu") (net 7))
+  (segment (start 183.0296 72.592) (end 188.102811 77.665211) (width 0.5) (layer "B.Cu") (net 7))
   (segment (start 198.78 113.592) (end 197.801 112.614) (width 0.5) (layer "B.Cu") (net 7))
+  (segment (start 187.127021 107.209021) (end 192.532 112.614) (width 0.5) (layer "B.Cu") (net 7))
   (segment (start 198.78 115.219) (end 198.78 113.592) (width 0.5) (layer "B.Cu") (net 7))
   (segment (start 207.9256 117.15) (end 204.4976 117.15) (width 0.5) (layer "B.Cu") (net 7))
-  (segment (start 197.801 112.614) (end 191.839 112.614) (width 0.5) (layer "B.Cu") (net 7))
-  (segment (start 185.127021 105.902021) (end 185.127021 104.8856) (width 0.5) (layer "B.Cu") (net 7))
+  (segment (start 187.031464 104.790043) (end 187.127021 104.8856) (width 0.5) (layer "B.Cu") (net 7))
+  (segment (start 187.127021 104.8856) (end 187.127021 107.209021) (width 0.5) (layer "B.Cu") (net 7))
+  (segment (start 188.102811 100.848753) (end 187.031464 101.9201) (width 0.5) (layer "B.Cu") (net 7))
+  (segment (start 187.031464 101.9201) (end 187.031464 104.790043) (width 0.5) (layer "B.Cu") (net 7))
   (segment (start 207.108 97.87) (end 199.831 97.87) (width 0.25) (layer "F.Cu") (net 19))
   (segment (start 193.6076 90.7637) (end 193.6076 90.47) (width 0.25) (layer "F.Cu") (net 19))
@@
   (segment (start 174.263 79.5566) (end 174.263 81.0802) (width 0.5) (layer "B.Cu") (net 32))
   (segment (start 180.0296 73.79) (end 174.263 79.5566) (width 0.5) (layer "B.Cu") (net 32))
+  (segment (start 159.746 114.59) (end 153.418 114.59) (width 0.25) (layer "B.Cu") (net 34))
   (segment (start 151.068 116.94) (end 151.068 117.32) (width 0.25) (layer "B.Cu") (net 34))
   (segment (start 149.508 117.13) (end 149.6976 116.9404) (width 0.25) (layer "B.Cu") (net 34))
-  (segment (start 159.746 114.59) (end 179.601868 94.734132) (width 0.25) (layer "B.Cu") (net 34))
   (segment (start 153.4176 119.6696) (end 153.4176 119.67) (width 0.25) (layer "B.Cu") (net 34))
   (segment (start 149.698 116.94) (end 151.068 116.94) (width 0.25) (layer "B.Cu") (net 34))
   (segment (start 149.6976 116.9404) (end 149.6976 116.94) (width 0.25) (layer "B.Cu") (net 34))
+  (segment (start 153.418 114.59) (end 153.4176 114.5904) (width 0.25) (layer "B.Cu") (net 34))
   (segment (start 146.6696 117.13) (end 146.67 117.13) (width 0.25) (layer "B.Cu") (net 34))
   (segment (start 149.6976 116.9404) (end 149.698 116.94) (width 0.25) (layer "B.Cu") (net 34))
-  (segment (start 153.418 114.59) (end 159.746 114.59) (width 0.25) (layer "B.Cu") (net 34))
   (segment (start 146.67 117.13) (end 149.508 117.13) (width 0.25) (layer "B.Cu") (net 34))
-  (segment (start 153.4176 114.5904) (end 153.418 114.59) (width 0.25) (layer "B.Cu") (net 34))
+  (segment (start 186.502811 94.734132) (end 179.601868 94.734132) (width 0.25) (layer "B.Cu") (net 34))
+  (segment (start 179.601868 94.734132) (end 159.746 114.59) (width 0.25) (layer "B.Cu") (net 34))
   (segment (start 151.068 116.94) (end 153.4176 114.5904) (width 0.25) (layer "B.Cu") (net 34))
   (segment (start 153.4176 119.6696) (end 153.418 119.67) (width 0.25) (layer "B.Cu") (net 34))
   (segment (start 151.068 117.32) (end 153.4176 119.6696) (width 0.25) (layer "B.Cu") (net 34))
   (segment (start 153.4176 114.5904) (end 153.4176 114.59) (width 0.25) (layer "B.Cu") (net 34))
-  (segment (start 179.601868 94.734132) (end 184.502811 94.734132) (width 0.25) (layer "B.Cu") (net 34))
   (zone (net 1) (net_name "GND") (layers "F&B.Cu") (name "GND") (hatch edge 0.508)
     (connect_pads (clearance 0.508))
