File: hardware/bGeigieZen V3.0.0/bGeigieZen V3.0.0.kicad_sch (KiCad schematic)
At the start: 24 parts, among them J1 M5 2x15 pin, J10 QI GND, J11 QI charger Plus, J2 Geiger, J3 GPS, J4 Geiger 2, J5 Extra support header, J6 Grove, J7 Grove, J8 QI charger ground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

Commit message: Updated, cleaned out old files
Parts:
- removed C1: 47uF, bGeigieNano V1.1.5:C025-024X044, symbol bGeigieRaku-V2-rescue:bGeigieNano_V1.1.5-eagle-import_C-EU025-024X044-bGeigieNa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
- removed H1, H10, H2, H3, H5, H7, H8, H9: MountingHole_Pad, MountingHole:MountingHole_3.2mm_M3, symbol Mechanical:MountingHole_Pad
Connections:
- net Reset: no longer names the net of J1.5 (Pin_5)
Other:
- moved on the sheet: H4, H6

Commit message: added board updates
Parts:
- J2: value Geiger -> Geiger IRover
- J4: value Geiger 2 -> Geiger Safepulse
Changed lines of the file:
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@@
       (effects (font (size 1.27 1.27)) (justify right))
     )
-    (property "Value" "Geiger" (at 196.85 66.04 0)
+    (property "Value" "Geiger IRover" (at 196.85 66.04 0)
       (effects (font (size 1.27 1.27)) (justify right))
     )
@@
       (effects (font (size 1.27 1.27)) (justify right))
     )
-    (property "Value" "Geiger 2" (at 196.85 56.515 0)
+    (property "Value" "Geiger Safepulse" (at 196.85 56.515 0)
       (effects (font (size 1.27 1.27)) (justify right))
     )

Commit message: Added draw.io and updated V3.0.0 board
Parts:
- J1: footprint Connector_PinHeader_2.54mm:PinHeader_2x15_P2.54mm_Vertical_SMD -> Connector_PinHeader_2.54mm:PinHeader_2x15_P2.54mm_Vertical
Changed lines of the file:
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@@
       (effects (font (size 1.27 1.27)))
     )
-    (property "Footprint" "Connector_PinHeader_2.54mm:PinHeader_2x15_P2.54mm_Vertical_SMD" (at 140.97 93.98 0)
+    (property "Footprint" "Connector_PinHeader_2.54mm:PinHeader_2x15_P2.54mm_Vertical" (at 140.97 93.98 0)
       (effects (font (size 1.27 1.27)) hide)
     )

Commit message: added grove connector for motion sensor
Parts:
- removed J7: Grove, Connector_JST:JST_ACH_BM04B-ACHSS-A-GAN-ETF_1x04-1MP_P1.20mm_Vertical, symbol 110990030:110990030
- J6: footprint Connector_JST:JST_ACH_BM04B-ACHSS-A-GAN-ETF_1x04-1MP_P1.20mm_Vertical -> Connector_PinSocket_2.00mm:PinSocket_1x04_P2.00mm_Horizontal

Commit message: Updated board for IMU and I2C
Connections:
- net 3.3V: now also J6.3; no longer J6.2
- net GND: now also J6.4; no longer J6.1
- net SCL: now also J6.1; no longer J6.3
- net SDA: now also J6.2; no longer J6.4
Changed lines of the file:
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@@
   (junction (at 125.73 125.73) (diameter 0.3048) (color 0 0 0 0)
   )
+  (junction (at 146.05 96.52) (diameter 0) (color 0 0 0 0)
+  )
   (junction (at 186.69 82.55) (diameter 0.3048) (color 0 0 0 0)
   )
@@
     (stroke (width 0) (type solid))
   )
-  (wire (pts (xy 184.15 95.25) (xy 181.61 95.25))
-    (stroke (width 0) (type default))
-  )
   (wire (pts (xy 130.81 78.74) (xy 133.35 78.74))
     (stroke (width 0) (type solid))
@@
     (stroke (width 0) (type solid))
   )
+  (wire (pts (xy 168.91 95.25) (xy 184.15 95.25))
+    (stroke (width 0) (type default))
+  )
   (wire (pts (xy 130.81 81.28) (xy 133.35 81.28))
     (stroke (width 0) (type solid))
@@
     (stroke (width 0) (type solid))
   )
+  (wire (pts (xy 146.05 96.52) (xy 168.91 96.52))
+    (stroke (width 0) (type default))
+  )
   (wire (pts (xy 189.23 66.04) (xy 185.42 66.04))
     (stroke (width 0) (type solid))
@@
     (stroke (width 0) (type solid))
   )
+  (wire (pts (xy 143.51 96.52) (xy 146.05 96.52))
+    (stroke (width 0) (type default))
+  )
   (wire (pts (xy 186.69 82.55) (xy 186.69 63.5))
     (stroke (width 0) (type solid))
@@
     (stroke (width 0) (type solid))
   )
-  (wire (pts (xy 167.64 100.33) (xy 167.64 96.52))
-    (stroke (width 0) (type default))
-  )
-  (wire (pts (xy 171.45 102.235) (xy 171.45 120.65))
-    (stroke (width 0) (type default))
-  )
   (wire (pts (xy 69.85 77.47) (xy 69.85 80.01))
     (stroke (width 0) (type solid))
@@
     (stroke (width 0) (type solid))
   )
-  (wire (pts (xy 180.34 97.79) (xy 184.15 97.79))
-    (stroke (width 0) (type default))
-  )
   (wire (pts (xy 113.03 78.74) (xy 116.84 78.74))
     (stroke (width 0) (type solid))
   )
+  (wire (pts (xy 182.88 97.79) (xy 184.15 97.79))
+    (stroke (width 0) (type default))
+  )
   (wire (pts (xy 170.18 80.01) (xy 170.18 119.38))
     (stroke (width 0) (type solid))
@@
     (stroke (width 0) (type solid))
   )
+  (wire (pts (xy 168.91 95.25) (xy 168.91 96.52))
+    (stroke (width 0) (type default))
+  )
   (wire (pts (xy 185.42 56.515) (xy 185.42 66.04))
     (stroke (width 0) (type solid))
@@
     (stroke (width 0) (type solid))
   )
-  (wire (pts (xy 180.34 102.235) (xy 180.34 97.79))
-    (stroke (width 0) (type default))
-  )
   (wire (pts (xy 172.72 82.55) (xy 172.72 125.73))
     (stroke (width 0) (type solid))
@@
     (stroke (width 0) (type solid))
   )
-  (wire (pts (xy 171.45 102.235) (xy 180.34 102.235))
+  (wire (pts (xy 171.45 92.71) (xy 184.15 92.71))
     (stroke (width 0) (type default))
   )
@@
     (stroke (width 0) (type solid))
   )
-  (wire (pts (xy 181.61 88.265) (xy 181.61 95.25))
-    (stroke (width 0) (type default))
-  )
-  (wire (pts (xy 167.64 100.33) (xy 184.15 100.33))
-    (stroke (width 0) (type default))
-  )
   (wire (pts (xy 166.37 74.93) (xy 166.37 88.9))
     (stroke (width 0) (type default))
@@
     (stroke (width 0) (type solid))
   )
-  (wire (pts (xy 146.05 96.52) (xy 167.64 96.52))
-    (stroke (width 0) (type default))
-  )
   (wire (pts (xy 146.05 106.68) (xy 153.035 106.68))
     (stroke (width 0) (type default))
@@
   (wire (pts (xy 120.65 66.04) (xy 151.765 66.04))
     (stroke (width 0) (type solid))
+  )
+  (wire (pts (xy 171.45 92.71) (xy 171.45 120.65))
+    (stroke (width 0) (type default))
   )
   (text "QI charger LIPO minus" (exclude_from_sim no)
@@
     (effects (font (size 1.27 1.27) (color 56 88 62 1)) (justify left bottom))
   )
-  (label "SDA" (at 149.86 96.52 0) (fields_autoplaced)
+  (label "SDA" (at 147.32 96.52 0) (fields_autoplaced)
     (effects (font (size 1.27 1.27)) (justify right bottom))
   )
@@
     (effects (font (size 1.27 1.27)) (justify left bottom))
   )
-  (label "SCL" (at 184.15 97.79 0) (fields_autoplaced)
+  (label "SCL" (at 184.15 92.71 0) (fields_autoplaced)
     (effects (font (size 1.27 1.27)) (justify right bottom))
   )
@@
     (effects (font (size 1.27 1.27)) (justify left bottom))
   )
-  (label "SDA" (at 184.15 100.33 0) (fields_autoplaced)
+  (label "SDA" (at 181.61 95.25 0) (fields_autoplaced)
     (effects (font (size 1.27 1.27)) (justify right bottom))
   )
-  (global_label "3.3V" (shape bidirectional) (at 181.61 88.265 180)
+  (global_label "3.3V" (shape bidirectional) (at 182.88 97.79 180)
     (effects (font (size 1.27 1.27)) (justify right))
-    (property "Intersheetrefs" "${INTERSHEET_REFS}" (at 20.32 13.335 0)
+    (property "Intersheetrefs" "${INTERSHEET_REFS}" (at 21.59 22.86 0)
       (effects (font (size 1.27 1.27)) hide)
     )
@@
     )
   )
-  (symbol (lib_id "bGeigieRaku-V2-rescue:GND-bGeigieNano_V1.1.5") (at 184.15 90.17 180) (unit 1)
-    (exclude_from_sim no) (in_bom yes) (on_board yes) (dnp no)
-    (property "Reference" "#GND0102" (at 184.15 90.17 0)
-      (effects (font (size 1.27 1.27)) hide)
-    )
-    (property "Value" "GND" (at 184.15 87.0966 0)
+  (symbol (lib_id "bGeigieRaku-V2-rescue:GND-bGeigieNano_V1.1.5") (at 184.15 102.87 0) (unit 1)
+    (exclude_from_sim no) (in_bom yes) (on_board yes) (dnp no)
+    (property "Reference" "#GND0102" (at 184.15 102.87 0)
+      (effects (font (size 1.27 1.27)) hide)
+    )
+    (property "Value" "GND" (at 184.15 105.9434 0)
       (effects (font (size 1.4986 1.4986)))
     )
-    (property "Footprint" "" (at 184.15 90.17 0)
-      (effects (font (size 1.27 1.27)) hide)
-    )
-    (property "Datasheet" "" (at 184.15 90.17 0)
-      (effects (font (size 1.27 1.27)) hide)
-    )
-    (property "Description" "" (at 184.15 90.17 0)
-      (effects (font (size 1.27 1.27)) hide)
-    )
+    (property "Footprint" "" (at 184.15 102.87 0)
+      (effects (font (size 1.27 1.27)) hide)
+    )
+    (property "Datasheet" "" (at 184.15 102.87 0)
+      (effects (font (size 1.27 1.27)) hide)
+    )
+    (property "Description" "" (at 184.15 102.87 0)
+      (effects (font (size 1.27 1.27)) hide)
+    )

Commit message: Updated Grove connector on board V3.0.1
Connections:
- net 3.3V: now also J6.2; no longer J6.3
- net GND: now also J6.1; no longer J6.4
- net SCL: now also J6.4; no longer J6.1
- net SDA: now also J6.3; no longer J6.2
Changed lines of the file:
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@@
   (junction (at 125.73 125.73) (diameter 0.3048) (color 0 0 0 0)
   )
-  (junction (at 146.05 96.52) (diameter 0) (color 0 0 0 0)
-  )
   (junction (at 186.69 82.55) (diameter 0.3048) (color 0 0 0 0)
   )
@@
     (stroke (width 0) (type solid))
   )
+  (wire (pts (xy 171.45 100.33) (xy 184.15 100.33))
+    (stroke (width 0) (type default))
+  )
   (wire (pts (xy 135.89 125.73) (xy 172.72 125.73))
     (stroke (width 0) (type solid))
@@
     (stroke (width 0) (type solid))
   )
-  (wire (pts (xy 168.91 95.25) (xy 184.15 95.25))
-    (stroke (width 0) (type default))
-  )
   (wire (pts (xy 130.81 81.28) (xy 133.35 81.28))
     (stroke (width 0) (type solid))
@@
     (stroke (width 0) (type default))
   )
+  (wire (pts (xy 177.8 88.9) (xy 184.15 88.9))
+    (stroke (width 0) (type default))
+  )
   (wire (pts (xy 72.39 85.09) (xy 72.39 106.045))
     (stroke (width 0) (type default))
@@
     (stroke (width 0) (type solid))
   )
-  (wire (pts (xy 143.51 96.52) (xy 146.05 96.52))
-    (stroke (width 0) (type default))
-  )
   (wire (pts (xy 186.69 82.55) (xy 186.69 63.5))
     (stroke (width 0) (type solid))
@@
     (stroke (width 0) (type solid))
   )
+  (wire (pts (xy 184.15 88.9) (xy 184.15 92.71))
+    (stroke (width 0) (type default))
+  )
   (wire (pts (xy 133.35 104.14) (xy 131.445 104.14))
     (stroke (width 0) (type default))
@@
     (stroke (width 0) (type solid))
   )
+  (wire (pts (xy 180.34 95.25) (xy 184.15 95.25))
+    (stroke (width 0) (type default))
+  )
   (wire (pts (xy 113.03 78.74) (xy 116.84 78.74))
     (stroke (width 0) (type solid))
   )
-  (wire (pts (xy 182.88 97.79) (xy 184.15 97.79))
+  (wire (pts (xy 168.91 97.79) (xy 184.15 97.79))
+    (stroke (width 0) (type default))
+  )
+  (wire (pts (xy 171.45 100.33) (xy 171.45 120.65))
     (stroke (width 0) (type default))
   )
@@
     (stroke (width 0) (type solid))
   )
-  (wire (pts (xy 168.91 95.25) (xy 168.91 96.52))
+  (wire (pts (xy 168.91 97.79) (xy 168.91 96.52))
     (stroke (width 0) (type default))
   )
@@
     (stroke (width 0) (type solid))
   )
-  (wire (pts (xy 171.45 92.71) (xy 184.15 92.71))
-    (stroke (width 0) (type default))
-  )
   (wire (pts (xy 166.37 74.93) (xy 184.15 74.93))
     (stroke (width 0) (type solid))
@@
   (wire (pts (xy 120.65 66.04) (xy 151.765 66.04))
     (stroke (width 0) (type solid))
-  )
-  (wire (pts (xy 171.45 92.71) (xy 171.45 120.65))
-    (stroke (width 0) (type default))
   )
   (text "QI charger LIPO minus" (exclude_from_sim no)
@@
     (effects (font (size 1.27 1.27) (color 56 88 62 1)) (justify left bottom))
   )
-  (label "SDA" (at 147.32 96.52 0) (fields_autoplaced)
+  (label "SDA" (at 151.13 96.52 180) (fields_autoplaced)
     (effects (font (size 1.27 1.27)) (justify right bottom))
   )
-  (label "TX2" (at 133.35 93.98 0) (fields_autoplaced)
+  (label "TX2" (at 133.35 93.98 180) (fields_autoplaced)
     (effects (font (size 1.27 1.27)) (justify right bottom))
   )
-  (label "VBATT" (at 100.965 76.2 0) (fields_autoplaced)
+  (label "VBATT" (at 100.965 76.2 180) (fields_autoplaced)
     (effects (font (size 1.27 1.27)) (justify right bottom))
   )
@@
     (effects (font (size 1.27 1.27)) (justify left bottom))
   )
-  (label "GIO2 on Core and GIO32 on Core-2" (at 133.35 99.06 0) (fields_autoplaced)
+  (label "GIO2 on Core and GIO32 on Core-2" (at 133.35 99.06 180) (fields_autoplaced)
     (effects (font (size 1.27 1.27)) (justify right bottom))
   )
@@
     (effects (font (size 1.27 1.27)) (justify left bottom))
   )
-  (label "SCL" (at 184.15 92.71 0) (fields_autoplaced)
+  (label "SCL" (at 184.15 100.33 180) (fields_autoplaced)
     (effects (font (size 1.27 1.27)) (justify right bottom))
   )
-  (label "SCL" (at 133.35 96.52 0) (fields_autoplaced)
+  (label "SCL" (at 133.35 96.52 180) (fields_autoplaced)
     (effects (font (size 1.27 1.27)) (justify right bottom))
   )
@@
     (effects (font (size 1.27 1.27)) (justify left bottom))
   )
-  (label "SDA" (at 181.61 95.25 0) (fields_autoplaced)
+  (label "SDA" (at 184.15 97.79 180) (fields_autoplaced)
     (effects (font (size 1.27 1.27)) (justify right bottom))
   )
-  (global_label "3.3V" (shape bidirectional) (at 182.88 97.79 180)
+  (global_label "3.3V" (shape bidirectional) (at 180.34 95.25 180)
     (effects (font (size 1.27 1.27)) (justify right))
-    (property "Intersheetrefs" "${INTERSHEET_REFS}" (at 21.59 22.86 0)
+    (property "Intersheetrefs" "${INTERSHEET_REFS}" (at 19.05 20.32 0)
       (effects (font (size 1.27 1.27)) hide)
     )
@@
     )
   )
-  (symbol (lib_id "bGeigieRaku-V2-rescue:GND-bGeigieNano_V1.1.5") (at 184.15 102.87 0) (unit 1)
-    (exclude_from_sim no) (in_bom yes) (on_board yes) (dnp no)
-    (property "Reference" "#GND0102" (at 184.15 102.87 0)
-      (effects (font (size 1.27 1.27)) hide)
-    )
-    (property "Value" "GND" (at 184.15 105.9434 0)
+  (symbol (lib_id "bGeigieRaku-V2-rescue:GND-bGeigieNano_V1.1.5") (at 177.8 91.44 0) (unit 1)
+    (exclude_from_sim no) (in_bom yes) (on_board yes) (dnp no)
+    (property "Reference" "#GND0102" (at 177.8 91.44 0)
+      (effects (font (size 1.27 1.27)) hide)
+    )
+    (property "Value" "GND" (at 181.61 93.218 0)
       (effects (font (size 1.4986 1.4986)))
     )
-    (property "Footprint" "" (at 184.15 102.87 0)
-      (effects (font (size 1.27 1.27)) hide)
-    )
-    (property "Datasheet" "" (at 184.15 102.87 0)
-      (effects (font (size 1.27 1.27)) hide)
-    )
-    (property "Description" "" (at 184.15 102.87 0)
-      (effects (font (size 1.27 1.27)) hide)
-    )
+    (property "Footprint" "" (at 177.8 91.44 0)
+      (effects (font (size 1.27 1.27)) hide)
+    )
+    (property "Datasheet" "" (at 177.8 91.44 0)
+      (effects (font (size 1.27 1.27)) hide)
+    )
+    (property "Description" "" (at 177.8 91.44 0)
+      (effects (font (size 1.27 1.27)) hide)
+    )

Commit message: Updated Version number to V3.0.1 on the boards
Other:
- title: bGeigieZen V2.1.2 -> bGeigieZen V3.0.1
Changed lines of the file:
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@@
   (paper "A4")
   (title_block
-    (title "bGeigieZen V2.1.2")
-    (date "2023-05-29")
-    (rev "V3.0.0")
+    (title "bGeigieZen V3.0.1")
+    (date "2023-10-04")
+    (rev "V3.0.3")
     (company "GitHub link at https://github.com/Safecast/bGeigieZen")
   )

Commit message: Updated board a bit more
Connections:
- net 3.3V: now also J6.3; no longer J6.2
- net GND: now also J6.4; no longer J6.1
- net SCL: now also J6.1; no longer J6.4
- net SDA: now also J6.2; no longer J6.3
Changed lines of the file:
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@@
   (title_block
     (title "bGeigieZen V3.0.1")
-    (date "2023-10-04")
-    (rev "V3.0.3")
+    (date "2023-10-28")
+    (rev "V3.0.1")
     (company "GitHub link at https://github.com/Safecast/bGeigieZen")
   )
   (junction (at 125.73 125.73) (diameter 0.3048) (color 0 0 0 0)
   )
+  (junction (at 146.05 96.52) (diameter 0) (color 0 0 0 0)
+  )
   (junction (at 186.69 82.55) (diameter 0.3048) (color 0 0 0 0)
   )
@@
     (stroke (width 0) (type solid))
   )
-  (wire (pts (xy 171.45 100.33) (xy 184.15 100.33))
-    (stroke (width 0) (type default))
-  )
   (wire (pts (xy 135.89 125.73) (xy 172.72 125.73))
     (stroke (width 0) (type solid))
@@
     (stroke (width 0) (type solid))
   )
+  (wire (pts (xy 168.91 95.25) (xy 184.15 95.25))
+    (stroke (width 0) (type default))
+  )
   (wire (pts (xy 130.81 81.28) (xy 133.35 81.28))
     (stroke (width 0) (type solid))
@@
     (stroke (width 0) (type default))
   )
-  (wire (pts (xy 177.8 88.9) (xy 184.15 88.9))
-    (stroke (width 0) (type default))
-  )
   (wire (pts (xy 72.39 85.09) (xy 72.39 106.045))
     (stroke (width 0) (type default))
@@
     (stroke (width 0) (type solid))
   )
+  (wire (pts (xy 143.51 96.52) (xy 146.05 96.52))
+    (stroke (width 0) (type default))
+  )
   (wire (pts (xy 186.69 82.55) (xy 186.69 63.5))
     (stroke (width 0) (type solid))
@@
     (stroke (width 0) (type solid))
   )
-  (wire (pts (xy 184.15 88.9) (xy 184.15 92.71))
-    (stroke (width 0) (type default))
-  )
   (wire (pts (xy 133.35 104.14) (xy 131.445 104.14))
     (stroke (width 0) (type default))
@@
     (stroke (width 0) (type solid))
   )
-  (wire (pts (xy 180.34 95.25) (xy 184.15 95.25))
-    (stroke (width 0) (type default))
-  )
   (wire (pts (xy 113.03 78.74) (xy 116.84 78.74))
     (stroke (width 0) (type solid))
   )
-  (wire (pts (xy 168.91 97.79) (xy 184.15 97.79))
-    (stroke (width 0) (type default))
-  )
-  (wire (pts (xy 171.45 100.33) (xy 171.45 120.65))
+  (wire (pts (xy 182.88 97.79) (xy 184.15 97.79))
     (stroke (width 0) (type default))
   )
@@
     (stroke (width 0) (type solid))
   )
-  (wire (pts (xy 168.91 97.79) (xy 168.91 96.52))
+  (wire (pts (xy 168.91 95.25) (xy 168.91 96.52))
     (stroke (width 0) (type default))
   )
@@
     (stroke (width 0) (type solid))
   )
+  (wire (pts (xy 171.45 92.71) (xy 184.15 92.71))
+    (stroke (width 0) (type default))
+  )
   (wire (pts (xy 166.37 74.93) (xy 184.15 74.93))
     (stroke (width 0) (type solid))
@@
   (wire (pts (xy 120.65 66.04) (xy 151.765 66.04))
     (stroke (width 0) (type solid))
+  )
+  (wire (pts (xy 171.45 92.71) (xy 171.45 120.65))
+    (stroke (width 0) (type default))
   )
   (text "QI charger LIPO minus" (exclude_from_sim no)
@@
     (effects (font (size 1.27 1.27) (color 56 88 62 1)) (justify left bottom))
   )
-  (label "SDA" (at 151.13 96.52 180) (fields_autoplaced)
+  (label "SDA" (at 147.32 96.52 180) (fields_autoplaced)
     (effects (font (size 1.27 1.27)) (justify right bottom))
   )
@@
     (effects (font (size 1.27 1.27)) (justify left bottom))
   )
-  (label "SCL" (at 184.15 100.33 180) (fields_autoplaced)
+  (label "SCL" (at 184.15 92.71 180) (fields_autoplaced)
     (effects (font (size 1.27 1.27)) (justify right bottom))
   )
@@
     (effects (font (size 1.27 1.27)) (justify left bottom))
   )
-  (label "SDA" (at 184.15 97.79 180) (fields_autoplaced)
+  (label "SDA" (at 181.61 95.25 180) (fields_autoplaced)
     (effects (font (size 1.27 1.27)) (justify right bottom))
   )
-  (global_label "3.3V" (shape bidirectional) (at 180.34 95.25 180)
+  (global_label "3.3V" (shape bidirectional) (at 182.88 97.79 180)
     (effects (font (size 1.27 1.27)) (justify right))
-    (property "Intersheetrefs" "${INTERSHEET_REFS}" (at 19.05 20.32 0)
+    (property "Intersheetrefs" "${INTERSHEET_REFS}" (at 21.59 22.86 0)
       (effects (font (size 1.27 1.27)) hide)
     )
@@
     )
   )
-  (symbol (lib_id "bGeigieRaku-V2-rescue:GND-bGeigieNano_V1.1.5") (at 177.8 91.44 0) (unit 1)
-    (exclude_from_sim no) (in_bom yes) (on_board yes) (dnp no)
-    (property "Reference" "#GND0102" (at 177.8 91.44 0)
-      (effects (font (size 1.27 1.27)) hide)
-    )
-    (property "Value" "GND" (at 181.61 93.218 0)
+  (symbol (lib_id "bGeigieRaku-V2-rescue:GND-bGeigieNano_V1.1.5") (at 184.15 102.87 0) (unit 1)
+    (exclude_from_sim no) (in_bom yes) (on_board yes) (dnp no)
+    (property "Reference" "#GND0102" (at 184.15 102.87 0)
+      (effects (font (size 1.27 1.27)) hide)
+    )
+    (property "Value" "GND" (at 184.15 105.9434 0)
       (effects (font (size 1.4986 1.4986)))
     )
-    (property "Footprint" "" (at 177.8 91.44 0)
-      (effects (font (size 1.27 1.27)) hide)
-    )
-    (property "Datasheet" "" (at 177.8 91.44 0)
-      (effects (font (size 1.27 1.27)) hide)
-    )
-    (property "Description" "" (at 177.8 91.44 0)
-      (effects (font (size 1.27 1.27)) hide)
-    )
+    (property "Footprint" "" (at 184.15 102.87 0)
+      (effects (font (size 1.27 1.27)) hide)
+    )
+    (property "Datasheet" "" (at 184.15 102.87 0)
+      (effects (font (size 1.27 1.27)) hide)
+    )
+    (property "Description" "" (at 184.15 102.87 0)
+      (effects (font (size 1.27 1.27)) hide)
+    )
