File: hardware/bGeigieZen 3.0.1 production/bGeigieZen 3.0.1 production.kicad_sch (KiCad schematic)
At the start: 14 parts, among them J1 M5 2x15 pin, J10 QI GND, J11 QI charger Plus, J2 Geiger IRover, J3 GPS, J4 Geiger Safepulse, J5 Extra support header, J6 Grove, J8 QI charger ground, J9 QI Plus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

Commit message: Update Board to V3.0.2 (adjusted placement of the 4056)
Other:
- title: bGeigieZen V3.0.1 -> bGeigieZen V3.0.2
Changed lines of the file:
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@@
 	(version 20231120)
 	(generator "eeschema")
-	(generator_version "7.99")
+	(generator_version "8.0")
 	(paper "A4")
 	(title_block
-		(title "bGeigieZen V3.0.1")
-		(date "2023-10-28")
-		(rev "V3.0.1")
+		(title "bGeigieZen V3.0.2")
+		(date "2024-01-17")
+		(rev "V3.0.2")
 		(company "GitHub link at https://github.com/Safecast/bGeigieZen")
 	)
@@
 		)
 		(instances
-			(project "bGeigieZen V3.0.0"
+			(project "bGeigieZen 3.0.1 production"
 				(path "/c2e3a215-6a49-419d-95d1-595f35b17280"
 					(reference "J1")
@@
 		)
 		(instances
-			(project "bGeigieZen V3.0.0"
+			(project "bGeigieZen 3.0.1 production"
 				(path "/c2e3a215-6a49-419d-95d1-595f35b17280"
 					(reference "BT1")
@@
 		)
 		(instances
-			(project "bGeigieZen V3.0.0"
+			(project "bGeigieZen 3.0.1 production"
 				(path "/c2e3a215-6a49-419d-95d1-595f35b17280"
 					(reference "J3")
@@
 		)
 		(instances
-			(project "bGeigieZen V3.0.0"
+			(project "bGeigieZen 3.0.1 production"
 				(path "/c2e3a215-6a49-419d-95d1-595f35b17280"
 					(reference "SW1")
@@
 		)
 		(instances
-			(project "bGeigieZen V3.0.0"
+			(project "bGeigieZen 3.0.1 production"
 				(path "/c2e3a215-6a49-419d-95d1-595f35b17280"
 					(reference "J2")
@@
 		)
 		(instances
-			(project "bGeigieZen V3.0.0"
+			(project "bGeigieZen 3.0.1 production"
 				(path "/c2e3a215-6a49-419d-95d1-595f35b17280"
 					(reference "#GND01")
@@
 		)
 		(instances
-			(project "bGeigieZen V3.0.0"
+			(project "bGeigieZen 3.0.1 production"
 				(path "/c2e3a215-6a49-419d-95d1-595f35b17280"
 					(reference "J11")
@@
 		)
 		(instances
-			(project "bGeigieZen V3.0.0"
+			(project "bGeigieZen 3.0.1 production"
 				(path "/c2e3a215-6a49-419d-95d1-595f35b17280"
 					(reference "J10")
@@
 		)
 		(instances
-			(project "bGeigieZen V3.0.0"
+			(project "bGeigieZen 3.0.1 production"
 				(path "/c2e3a215-6a49-419d-95d1-595f35b17280"
 					(reference "J9")
@@
 		)
 		(instances
-			(project "bGeigieZen V3.0.0"
+			(project "bGeigieZen 3.0.1 production"
 				(path "/c2e3a215-6a49-419d-95d1-595f35b17280"
 					(reference "H4")
@@
 		)
 		(instances
-			(project "bGeigieZen V3.0.0"
+			(project "bGeigieZen 3.0.1 production"
 				(path "/c2e3a215-6a49-419d-95d1-595f35b17280"
 					(reference "H6")
@@
 		)
 		(instances
-			(project "bGeigieZen V3.0.0"
+			(project "bGeigieZen 3.0.1 production"
 				(path "/c2e3a215-6a49-419d-95d1-595f35b17280"
 					(reference "J4")
@@
 		)
 		(instances
-			(project "bGeigieZen V3.0.0"
+			(project "bGeigieZen 3.0.1 production"
 				(path "/c2e3a215-6a49-419d-95d1-595f35b17280"
 					(reference "#GND0101")
@@
 		)
 		(instances
-			(project "bGeigieZen V3.0.0"
+			(project "bGeigieZen 3.0.1 production"
 				(path "/c2e3a215-6a49-419d-95d1-595f35b17280"
 					(reference "#GND0102")
@@
 		)
 		(instances
-			(project "bGeigieZen V3.0.0"
+			(project "bGeigieZen 3.0.1 production"
 				(path "/c2e3a215-6a49-419d-95d1-595f35b17280"
 					(reference "J6")
@@
 		)
 		(instances
-			(project "bGeigieZen V3.0.0"
+			(project "bGeigieZen 3.0.1 production"
 				(path "/c2e3a215-6a49-419d-95d1-595f35b17280"
 					(reference "J8")
@@
 		)
 		(instances
-			(project "bGeigieZen V3.0.0"
+			(project "bGeigieZen 3.0.1 production"
 				(path "/c2e3a215-6a49-419d-95d1-595f35b17280"
 					(reference "J5")
