File: hardware/bGeigieZen V4.x.x draft/bGeigieZen V4.x.x draft/bGeigieZen V4.x.x draft.kicad_sch (KiCad schematic)
At the start: 10 parts, among them J1 M5 2x15 pin, J2 Geiger IRover, J3 GPS, J4 Geiger Safepulse, J5 Extra support header, J6 Grove

Commit message: V4.0.3 boards
Other:
- title: bGeigieZen V4.0.2 -> bGeigieZen V4.0.3
Changed lines of the file:
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@@
 	(paper "A4")
 	(title_block
-		(title "bGeigieZen V4.0.2")
-		(date "2024-03-16")
-		(rev "V4.0.2")
+		(title "bGeigieZen V4.0.3")
+		(date "2024-03-25")
+		(rev "V4.0.3")
 		(company "GitHub link at https://github.com/Safecast/bGeigieZen")
 	)

Commit message: Changed the 18650 battery holder to a 1043 Keystone and modified the layout.
Parts:
- added J11: QI input +5V, Connector_PinHeader_2.54mm:PinHeader_1x01_P2.54mm_Vertical, symbol Connector:Conn_01x01_Pin
- added J7: QI GND out, Connector_PinHeader_2.54mm:PinHeader_1x01_P2.54mm_Vertical, symbol Connector:Conn_01x01_Pin
- added J8: QI input GND, Connector_PinHeader_2.54mm:PinHeader_1x01_P2.54mm_Vertical, symbol Connector:Conn_01x01_Pin
- added J9: QI battery out, Connector_PinHeader_2.54mm:PinHeader_1x01_P2.54mm_Vertical, symbol Connector:Conn_01x01_Pin
Connections:
- net BAT: now also J9.1 (Pin_1)
- net GND: now also J7.1 (Pin_1), J8.1 (Pin_1)
