File: hardware/bGeigieZen V4.x.x draft/bGeigieZen V4.x.x dual batteries 18500/bGeigieZen V4.x.x dual batteries 18500.kicad_pcb (KiCad board)
At the start: 2 copper layers, 129.4 x 64.6 mm, 16 parts, among them J1 M5 2x15 pin, J11 QI input +5V, J2 Geiger IRover, J3 GPS, J4 Geiger Safepulse, J5 Extra support header, J6 Grove, J7 QI GND out, J8 QI input GND, J9 QI battery out

Commit message: Updated V4.0.5 board with dual batteries
Parts:
- moved J8 56.6 mm to (209.3, 88.9)
- moved J7 56.6 mm to (181.6, 88.3)
- moved J9 56.6 mm to (181.8, 107.0)
- moved J11 56.6 mm to (209.6, 107.0)
- moved G front 42.3 mm to (178.4, 125.7), turned to 180 degrees
- moved J3 39.7 mm to (146.0, 104.0)
Routing:
- net /TX2: track 82.0 -> 38.9 mm, vias 1 -> 0
- net /RX2: track 81.4 -> 38.4 mm, vias 1 -> 0
- net /SDA: track 92.8 -> 57.1 mm, vias 0 -> 1
- net /SCL: track 103.0 -> 82.4 mm
- net /BAT: track 174.8 -> 162.4 mm
- net 3.3V: track 117.9 -> 125.0 mm

Commit message: Updated V4.0.3 boards
Parts:
- added G***: LOGO, bGeigieRaku_M5_1015:18650 map, B.Cu at (177.7, 120.4)
- added G***: LOGO, bGeigieRaku_M5_1015:18650 map, B.Cu at (178.0, 77.2)
- moved H4 6.30 mm to (99.4, 76.7)
- moved J1 6.30 mm to (139.2, 115.3)
- moved H6 6.30 mm to (99.5, 120.5)
- moved J3 5.75 mm to (151.7, 104.8)
Routing:
- net /BAT: track 162.4 -> 172.8 mm
- net 3.3V: track 125.0 -> 116.7 mm
- net /SCL: track 82.4 -> 74.3 mm
- net /GIO2 on Core and GIO32 on Core-2: track 115.6 -> 111.5 mm
- net /SDA: track 57.1 -> 58.1 mm, vias 1 -> 0
