File: hardware/bGeigieZen V4.x.x draft and production/bGeigieZen V4.x.x dual batteries 18500/bGeigieZen V4.x.x dual batteries 18500.kicad_pcb (KiCad board)
At the start: 2 copper layers, 129.4 x 64.6 mm, 12 parts, among them J1 M5 2x15 pin, J2 Geiger IRover, J3 GPS, J4 Geiger Safepulse, J5 Extra support header, J6 Grove

Commit message: Updated  boards to V4.0.4
Parts:
- removed J6: Grove, Connector_PinSocket_2.00mm:PinSocket_1x04_P2.00mm_Horizontal
Routing:
- net /SCL: track 69.2 -> 46.0 mm
- net 3.3V: track 113.3 -> 96.1 mm
- net /SDA: track 54.9 -> 38.7 mm
- net /RX2: track 39.3 -> 41.5 mm
- net /TX2: track 39.8 -> 41.9 mm
Other:
- board text added: "bGeigieZen V4.0.4 Production"
- board text removed: "bGeigieZen V4.0.3 Production"
