File: hardware/bGeigieZen V4.x.x draft and production/bGeigieZen V4.x.x single 18650/bGeigieZen V4.x.x single 18650.kicad_sch (KiCad schematic)
At the start: 11 parts, among them J1 M5 2x15 pin, J2 Geiger IRover, J3 GPS, J4 Geiger Safepulse, J5 Extra support header, SW1 SW_SPDT

Commit message: Added Zen stickers and Safecast drive 0.5.0 app
Parts:
- BT1: value 3.7 V Lipo -> 3.7 V Lipo
Other:
- title: bGeigieZen V4.0.5 -> bGeigieZen V4.0.6
Changed lines of the file:
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@@
 	(paper "A4")
 	(title_block
-		(title "bGeigieZen V4.0.5")
-		(date "2024-06-07")
+		(title "bGeigieZen V4.0.6")
+		(date "2024-06-29")
 		(rev "V4.0.5")
 		(company "GitHub link at https://github.com/Safecast/bGeigieZen")
@@
 			)
 		)
-		(property "Value" " 3.7 V Lipo"
+		(property "Value" "3.7 V Lipo"
 			(at 47.5075 92.2843 0)
 			(effects

Commit message: Updated boards for Zen V4.0.7
Other:
- title: bGeigieZen V4.0.6 -> bGeigieZen V4.0.7
Changed lines of the file:
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@@
 	(paper "A4")
 	(title_block
-		(title "bGeigieZen V4.0.6")
-		(date "2024-06-29")
-		(rev "V4.0.5")
+		(title "bGeigieZen V4.0.7")
+		(date "2024-07-07")
+		(rev "V4.0.7")
 		(company "GitHub link at https://github.com/Safecast/bGeigieZen")
 	)

Commit message: Updated boards to V4.0.8 and removed protected LiPo mounting holes.
Other:
- title: bGeigieZen V4.0.7 -> bGeigieZen V4.0.8
Changed lines of the file:
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@@
 	(paper "A4")
 	(title_block
-		(title "bGeigieZen V4.0.7")
-		(date "2024-08-14")
-		(rev "V4.0.7")
+		(title "bGeigieZen V4.0.8")
+		(date "2024-08-25")
+		(rev "V4.0.8")
 		(company "GitHub link at https://github.com/Safecast/bGeigieZen")
 	)

Commit message: On schematic too
Other:
- title: bGeigieZen V4.0.8 -> bGeigieZen V4.1.0 Standard
Changed lines of the file:
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@@
 	(paper "A4")
 	(title_block
-		(title "bGeigieZen V4.0.8")
-		(date "2024-08-25")
-		(rev "V4.0.8")
+		(title "bGeigieZen V4.1.0 Standard")
+		(date "2024-12-02")
+		(rev "V4.1.0")
 		(company "GitHub link at https://github.com/Safecast/bGeigieZen")
 	)
