File: hardware/bGeigieZen V4.x.x draft and production/bGeigieZen V4.x.x single 18650 rob/bGeigieZen V4.x.x single 18650 rob.kicad_sch (KiCad schematic)
At the start: 10 parts, among them J1 M5 2x15 pin, J3 GPS, J4 Geiger Safepulse, J5 Extra support header

Commit message: Rerouted the traces and made V4.0.8 NFW
Other:
- title: bGeigieZen V4.0.7 NFW -> bGeigieZen V4.0.8 NFW
Changed lines of the file:
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@@
 	(paper "A4")
 	(title_block
-		(title "bGeigieZen V4.0.7 NFW")
-		(date "2024-08-14")
-		(rev "V4.0.7 NFW")
+		(title "bGeigieZen V4.0.8 NFW")
+		(date "2024-09-23")
+		(rev "V4.0.8 NFW")
 		(company "GitHub link at https://github.com/Safecast/bGeigieZen")
 		(comment 1 "Not For Whimps version")

Commit message: Updated V4.1.0 NFW board an schematic.
Other:
- title: bGeigieZen V4.0.8 NFW -> bGeigieZen V4.1.0 NFW
Changed lines of the file:
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@@
 	(paper "A4")
 	(title_block
-		(title "bGeigieZen V4.0.8 NFW")
-		(date "2024-09-23")
-		(rev "V4.0.8 NFW")
+		(title "bGeigieZen V4.1.0 NFW")
+		(date "2024-12-02")
+		(rev "V4.1.0 NFW")
 		(company "GitHub link at https://github.com/Safecast/bGeigieZen")
 		(comment 1 "Not For Whimps version")
