File: hardware/bGeigieZen V4.x.x draft and production/bGeigieZen V4.x.x single 18650 rob/bGeigieZen V4.x.x single 18650 rob.kicad_pcb (KiCad board)
At the start: 2 copper layers, 129.4 x 64.6 mm, 13 parts, among them J1 M5 2x15 pin, J3 GPS, J4 Geiger Safepulse, J5 Extra support header

Commit message: Updated ground fills for NFW and standard boards
Parts:
- moved G*** 0.87 mm to (168.5, 77.5)
Changed lines of the file:
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@@
 	(footprint "bGeigieRaku_M5_1015:18650 map"
 		(layer "B.Cu")
-		(at 169.2808 77.9218 -90)
+		(at 168.5021 77.53 -90)
 		(property "Reference" "G***"
 			(at 0 0 90)
@@
 		(net 0)
 		(net_name "")
-		(layer "B.Cu")
+		(layers "F&B.Cu")
 		(hatch full 0.5)
 		(connect_pads
@@
 			(vias not_allowed)
 			(pads not_allowed)
-			(copperpour allowed)
+			(copperpour not_allowed)
 			(footprints allowed)
 		)
@@
 		(polygon
 			(pts
-				(xy 195.3076 70.03) (xy 210.8076 70.03) (xy 210.8076 81.53) (xy 207.3076 81.53) (xy 207.3076 83.03)
-				(xy 207.3076 92.03) (xy 201.8076 92.03) (xy 201.8076 83.03) (xy 195.3076 83.03)
+				(xy 195.3076 70.03) (xy 210.8076 70.03) (xy 210.8076 83.53) (xy 207.3076 83.53) (xy 207.3076 84.53)
+				(xy 207.3076 92.03) (xy 201.8076 92.03) (xy 201.8076 84.03) (xy 195.3076 84.03)
 			)
 		)

Commit message: Updated V4.1.1 NFW board
Other:
- board text added: "bGeigieZen V4.1.1 NFW"
- board text removed: "bGeigieZen V4.1.0 NFW"
Changed lines of the file:
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@@
 	(paper "A4")
 	(title_block
-		(title "bGeigieZenV4.1.0 NFW")
-		(date "2024-12-02")
-		(rev "V4.1.0")
+		(title "bGeigieZenV4.1.1 NFW")
+		(date "2025-03-03")
+		(rev "V4.1.1")
 		(comment 1 "Not For Whimps version.")
 	)
@@
 		(layer "Edge.Cuts")
 	)
-	(gr_text "bGeigieZen\nV4.1.0 NFW"
+	(gr_text "bGeigieZen\nV4.1.1 NFW"
 		(at 200.5584 112.724 90)
 		(layer "B.SilkS")
@@
 		)
 	)
-	(gr_text "bGeigieZen\nV4.1.0 NFW"
+	(gr_text "bGeigieZen\nV4.1.1 NFW"
 		(at 163.9316 124.2048 90)
 		(layer "F.SilkS")
@@
 		(polygon
 			(pts
-				(xy 195.3076 70.03) (xy 210.8076 70.03) (xy 210.8076 83.53) (xy 207.3076 83.53) (xy 207.3076 84.53)
+				(xy 195.3076 70.03) (xy 214.8076 70.03) (xy 214.8076 83.53) (xy 207.3076 83.53) (xy 207.3076 84.53)
 				(xy 207.3076 92.03) (xy 201.8076 92.03) (xy 201.8076 84.03) (xy 195.3076 84.03)
 			)

Commit message: Test CPU frequency change
Other:
- board text added: "+"
- board text added: "-"
- board text added: "GND"
- board text added: "RX"
- board text added: "TX"
Changed lines of the file:
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@@
+		)
+	)
+	(gr_text "+"
+		(at 191.77 96.976254 0)
+		(layer "F.SilkS")
+		(effects
+			(font
+				(size 1.5 1.5)
+				(thickness 0.3)
+				(bold yes)
+			)
+			(justify left bottom)
 		)
 	)
@@
 		)
 	)
+	(gr_text "TX"
+		(at 198.4756 97.23 90)
+		(layer "F.SilkS")
+		(effects
+			(font
+				(size 1.25 1.25)
+				(thickness 0.25)
+				(bold yes)
+			)
+			(justify left bottom)
+		)
+	)
 	(gr_text "M5StackCore"
 		(at 129.8956 101.814387 90)
@@
 		)
 	)
+	(gr_text "GND"
+		(at 200.9648 97.23 90)
+		(layer "F.SilkS")
+		(effects
+			(font
+				(size 1.25 1.25)
+				(thickness 0.25)
+				(bold yes)
+			)
+			(justify left bottom)
+		)
+	)
 	(gr_text "GPS"
 		(at 196.3076 85.53 90)
@@
 		)
 	)
+	(gr_text "RX"
+		(at 195.9864 97.373365 90)
+		(layer "F.SilkS")
+		(effects
+			(font
+				(size 1.25 1.25)
+				(thickness 0.25)
+				(bold yes)
+			)
+			(justify left bottom)
+		)
+	)
+	(gr_text "+"
+		(at 203.8096 96.5696 0)
+		(layer "B.SilkS")
+		(effects
+			(font
+				(size 1.5 1.5)
+				(thickness 0.3)
+				(bold yes)
+			)
+			(justify left bottom)
+		)
+	)
+	(gr_text "-"
+		(at 201.7776 96.5696 0)
+		(layer "B.SilkS")
+		(effects
+			(font
+				(size 1.5 1.5)
+				(thickness 0.3)
+				(bold yes)
+			)
+			(justify left bottom)
+		)
+	)
