File: hardware/bGeigieZen V5.x.x/bGeigieZen NFW/bGeigieZen NFW.kicad_sch (KiCad schematic)
At the start: 10 parts, among them J1 M5 2x15 pin, J3 GPS, J4 Geiger Safepulse, J5 Extra support header

Commit message: Update V4.2.0 boards and V5.x.x. boards
Parts:
- added J2: GPS, Connector_PinSocket_2.54mm:PinSocket_1x04_P2.54mm_Vertical, symbol Connector:Conn_01x04_Pin
- J3: value GPS -> Notecard; footprint Connector_PinSocket_2.54mm:PinSocket_1x06_P2.54mm_Vertical -> Connector_PinSocket_2.54mm:PinSocket_1x04_P2.54mm_Vertical; symbol Connector:Conn_01x06_Male -> Connector:Conn_01x04_Pin
- renumbered QI-charger to QI-charger1
Connections:
- net 3.3V: now also J3.4 (Pin_4), J2.4 (Pin_4); no longer J3.5 (Pin_5)
- net GND: now also J3.1 (Pin_1), J2.1 (Pin_1); no longer J3.2 (Pin_2)
- net RX2: now also J3.3 (Pin_3), J2.3 (Pin_3); no longer J3.4 (Pin_4)
- net TX2: now also J3.2 (Pin_2), J2.2 (Pin_2); no longer J3.3 (Pin_3)
Other:
- title: bGeigieZen V4.1.0 NFW -> bGeigieZen V5.0.0
Changed lines of the file:
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@@
 (kicad_sch
-	(version 20240716)
+	(version 20250114)
 	(generator "eeschema")
-	(generator_version "8.99")
+	(generator_version "9.0")
 	(paper "A4")
 	(title_block
-		(title "bGeigieZen V4.1.0 NFW")
-		(date "2024-12-02")
-		(rev "V4.1.0 NFW")
+		(title "bGeigieZen V5.0.0")
+		(date "2025-07-28")
+		(rev "V5.0.0")
 		(company "GitHub link at https://github.com/Safecast/bGeigieZen")
-		(comment 1 "Not For Whimps version")
+		(comment 1 "For GPS or Notecard")
 	)
 	(junction
@@
 	)
 	(junction
+		(at 166.37 88.9)
+		(diameter 0)
+		(color 0 0 0 0)
+	)
+	(junction
 		(at 186.69 82.55)
 		(diameter 0.3048)
@@
 	)
 	(junction
+		(at 172.72 96.52)
+		(diameter 0)
+		(color 0 0 0 0)
+	)
+	(junction
 		(at 184.15 74.93)
 		(diameter 0.3048)
+		(color 0 0 0 0)
+	)
+	(junction
+		(at 168.91 93.98)
+		(diameter 0)
+		(color 0 0 0 0)
+	)
+	(junction
+		(at 182.88 80.01)
+		(diameter 0)
 		(color 0 0 0 0)
 	)
@@
 	(wire
 		(pts
+			(xy 182.88 80.01) (xy 182.88 93.98)
+		)
+		(stroke
+			(width 0)
+			(type solid)
+		)
+	)
+	(wire
+		(pts
 			(xy 130.81 78.74) (xy 133.35 78.74)
 		)
@@
 	(wire
 		(pts
+			(xy 179.07 91.44) (xy 189.23 91.44)
+		)
+		(stroke
+			(width 0)
+			(type solid)
+		)
+	)
+	(wire
+		(pts
 			(xy 161.29 74.93) (xy 166.37 74.93)
 		)
@@
 	(wire
 		(pts
+			(xy 168.91 93.98) (xy 179.07 93.98)
+		)
+		(stroke
+			(width 0)
+			(type solid)
+		)
+	)
+	(wire
+		(pts
 			(xy 93.98 86.36) (xy 93.98 88.9)
 		)
@@
 	(wire
 		(pts
+			(xy 182.88 80.01) (xy 170.18 80.01)
+		)
+		(stroke
+			(width 0)
+			(type solid)
+		)
+	)
+	(wire
+		(pts
 			(xy 125.73 125.73) (xy 125.73 81.28)
 		)
@@
 	(wire
 		(pts
+			(xy 182.88 93.98) (xy 189.23 93.98)
+		)
+		(stroke
+			(width 0)
+			(type solid)
+		)
+	)
+	(wire
+		(pts
 			(xy 186.69 59.055) (xy 186.69 82.55)
 		)
@@
 	(wire
 		(pts
+			(xy 179.07 93.98) (xy 179.07 91.44)
+		)
+		(stroke
+			(width 0)
+			(type solid)
+		)
+	)
+	(wire
+		(pts
 			(xy 187.96 53.975) (xy 187.96 68.58)
 		)
@@
 	(wire
 		(pts
+			(xy 172.72 96.52) (xy 172.72 125.73)
+		)
+		(stroke
+			(width 0)
+			(type solid)
+		)
+	)
+	(wire
+		(pts
 			(xy 107.95 85.09) (xy 107.95 88.9)
 		)
@@
 	(wire
 		(pts
-			(xy 172.72 82.55) (xy 172.72 125.73)
+			(xy 172.72 82.55) (xy 172.72 96.52)
 		)
 		(stroke
@@
 	(wire
 		(pts
+			(xy 166.37 88.9) (xy 189.23 88.9)
+		)
+		(stroke
+			(width 0)
+			(type solid)
+		)
+	)
+	(wire
+		(pts
 			(xy 128.27 119.38) (xy 128.27 93.98)
 		)
@@
 	(wire
 		(pts
+			(xy 172.72 96.52) (xy 189.23 96.52)
+		)
+		(stroke
+			(width 0)
+			(type default)
+		)
+	)
+	(wire
+		(pts
 			(xy 129.54 99.06) (xy 133.35 99.06)
 		)
@@
 	(wire
 		(pts
-			(xy 189.23 80.01) (xy 170.18 80.01)
+			(xy 189.23 80.01) (xy 182.88 80.01)
 		)
 		(stroke
@@
 	(label "TX2"
 		(at 133.35 93.98 180)
-		(fields_autoplaced yes)
 		(effects
 			(font
@@
 	(label "GIO13"
 		(at 146.05 101.6 0)
-		(fields_autoplaced yes)
 		(effects
 			(font
@@
 	(label "GIO34"
 		(at 146.05 106.68 0)
-		(fields_autoplaced yes)
 		(effects
 			(font
@@
 	(label "GIO2 on Core and GIO32 on Core-2"
 		(at 132.08 99.06 180)
-		(fields_autoplaced yes)
 		(effects
 			(font
@@
 	(label "3.3V"
 		(at 146.05 88.9 0)
-		(fields_autoplaced yes)
 		(effects
 			(font
@@
 	(label "GIO5"
 		(at 146.05 99.06 0)
-		(fields_autoplaced yes)
 		(effects
 			(font
@@
 	(label "BAT"
 		(at 146.05 111.76 0)
-		(fields_autoplaced yes)
 		(effects
 			(font
@@
 	(label "RX2"
 		(at 146.05 93.98 0)
-		(fields_autoplaced yes)
 		(effects
 			(font
@@
 	)
 	(symbol
-		(lib_id "Connector:Conn_01x06_Male")
+		(lib_id "Connector:Conn_01x04_Pin")
 		(at 194.31 80.01 180)
 		(unit 1)
@@
 			)
 		)
-		(property "Value" "GPS"
-			(at 201.295 79.375 0)
+		(property "Value" "Notecard"
+			(at 205.74 81.28 0)
 			(effects
 				(font
@@
 			)
 		)
-		(property "Footprint" "Connector_PinSocket_2.54mm:PinSocket_1x06_P2.54mm_Vertical"
+		(property "Footprint" "Connector_PinSocket_2.54mm:PinSocket_1x04_P2.54mm_Vertical"
 			(at 194.31 80.01 0)
 			(effects
@@
 			)
 		)
-		(property "Description" ""
+		(property "Description" "Generic connector, single row, 01x04, script generated"
 			(at 194.31 80.01 0)
 			(effects
@@
 		)
 		(pin "4"
-		)
-		(pin "5"
-		)
-		(pin "6"
 		)
 		(instances
@@
 	)
 	(symbol
+		(lib_id "Connector:Conn_01x04_Pin")
+		(at 194.31 93.98 180)
+		(unit 1)
+		(exclude_from_sim no)
+		(in_bom yes)
+		(on_board yes)
+		(dnp no)
+		(property "Reference" "J2"
+			(at 200.025 90.805 0)
+			(effects
+				(font
+					(size 1.27 1.27)
+				)
+				(justify left)
+			)
+		)
+		(property "Value" "GPS"
+			(at 205.74 95.25 0)
+			(effects
+				(font
+					(size 1.27 1.27)
+				)
+				(justify left)
+			)
+		)
+		(property "Footprint" "Connector_PinSocket_2.54mm:PinSocket_1x04_P2.54mm_Vertical"
+			(at 194.31 93.98 0)
+			(effects
+				(font
+					(size 1.27 1.27)
+				)
+				(hide yes)
+			)
+		)
+		(property "Datasheet" "~"
+			(at 194.31 93.98 0)
+			(effects
+				(font
+					(size 1.27 1.27)
+				)
+				(hide yes)
+			)
+		)
+		(property "Description" "Generic connector, single row, 01x04, script generated"
+			(at 194.31 93.98 0)
+			(effects
+				(font
+					(size 1.27 1.27)
+				)
+				(hide yes)
+			)
+		)
+		(pin "1"
+		)
+		(pin "2"
+		)
+		(pin "3"
+		)
+		(pin "4"
+		)
+		(instances
+			(project "bGeigieZen NFW"
+				(path "/c2e3a215-6a49-419d-95d1-595f35b17280"
+					(reference "J2")
+					(unit 1)
+				)
+			)
+		)
+	)
+	(symbol
 		(lib_id "Connector:Conn_01x02_Male")
 		(at 113.03 82.55 0)
@@
 		(on_board yes)
 		(dnp no)
-		(property "Reference" "QI-charger"
+		(property "Reference" "QI-charger1"
 			(at 114.3 83.82 0)
 			(effects
@@
 			(project "bGeigieZen V4.x.x single 18650"
 				(path "/c2e3a215-6a49-419d-95d1-595f35b17280"
-					(reference "QI-charger")
+					(reference "QI-charger1")
 					(unit 1)
 				)
