File: hardware/bGeigieZen V4.x.x draft and production/bGeigieZen V4.2.x/bGeigieZen V4.2.x.kicad_sch (KiCad schematic)
At the start: 10 parts, among them J1 M5 2x15 pin, J3 GPS, J4 Geiger Safepulse, J5 Extra support header

Commit message: Changed V4.2.x board labeling
Parts:
- J3: footprint Connector_PinSocket_2.54mm:PinSocket_1x06_P2.54mm_Vertical -> Connector_PinSocket_2.54mm:PinSocket_1x04_P2.54mm_Vertical; symbol Connector:Conn_01x06_Male -> Connector_Generic:Conn_01x04
- renumbered QI-charger to QI-charger1
Connections:
- net 3.3V: now also J3.4 (Pin_4); no longer J3.5 (Pin_5)
- net GND: now also J3.1 (Pin_1); no longer J3.2 (Pin_2)
- net RX2: now also J3.3 (Pin_3); no longer J3.4 (Pin_4)
- net TX2: now also J3.2 (Pin_2); no longer J3.3 (Pin_3)
Changed lines of the file:
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@@
 	)
 	(symbol
-		(lib_id "Connector:Conn_01x06_Male")
-		(at 194.31 80.01 180)
+		(lib_id "Connector_Generic:Conn_01x04")
+		(at 194.31 80.01 0)
+		(mirror x)
 		(unit 1)
 		(exclude_from_sim no)
@@
 		(dnp no)
 		(property "Reference" "J3"
-			(at 200.025 76.835 0)
+			(at 188.595 76.835 0)
 			(effects
 				(font
@@
 		)
 		(property "Value" "GPS"
-			(at 201.295 79.375 0)
+			(at 198.12 78.74 0)
 			(effects
 				(font
@@
 			)
 		)
-		(property "Footprint" "Connector_PinSocket_2.54mm:PinSocket_1x06_P2.54mm_Vertical"
+		(property "Footprint" "Connector_PinSocket_2.54mm:PinSocket_1x04_P2.54mm_Vertical"
 			(at 194.31 80.01 0)
 			(effects
@@
 			)
 		)
-		(property "Description" ""
+		(property "Description" "Generic connector, single row, 01x04, script generated (kicad-library-utils/schlib/autogen/connector/)"
 			(at 194.31 80.01 0)
 			(effects
@@
 		)
 		(pin "4"
-		)
-		(pin "5"
-		)
-		(pin "6"
 		)
 		(instances
@@
 		(on_board yes)
 		(dnp no)
-		(property "Reference" "QI-charger"
+		(property "Reference" "QI-charger1"
 			(at 114.3 83.82 0)
 			(effects
@@
 			(project "bGeigieZen V4.x.x single 18650"
 				(path "/c2e3a215-6a49-419d-95d1-595f35b17280"
-					(reference "QI-charger")
-					(unit 1)
-				)
+					(reference "QI-charger1")
+					(unit 1)
+				)

Commit message: feat: update PCB version to V4.2.1 and adjust QI charger connector position
Other:
- title: bGeigieZen V4.2.0 -> bGeigieZen V4.2.1
Changed lines of the file:
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@@
 	(paper "A4")
 	(title_block
-		(title "bGeigieZen V4.2.0")
-		(date "2025-07-19")
-		(rev "V4.2.0")
+		(title "bGeigieZen V4.2.1")
+		(date "2025-10-10")
+		(rev "V4.2.1")
 		(company "GitHub link at https://github.com/Safecast/bGeigieZen")
 		(comment 1 "New standard version")
